Commit message: aggiunta sonar

File: bluerov2/bluerov2_description/urdf/sensors.xacro (robot description, xacro)
@@ -19,6 +19,14 @@
   <!-- Mount a camera -->
   <xacro:bluerov_camera namespace="" parent_link="${namespace}/base_link" suffix="_front">
-    <origin xyz="0.2 0 0" rpy="0 ${pi/4} 0"/>
+    <origin xyz="0.22 0 0" rpy="0 ${50*pi/180} 0"/>
   </xacro:bluerov_camera>
+  <!-- DVL (TODO: aggiustare corrispondenza tra la posizione e i dati del sensore) -->
+  <xacro:teledyne_wayfinder_dvl_macro namespace="${namespace}" parent_link="${namespace}/base_link" inertial_reference_frame="world">
+    <origin xyz="0 0 -0.05" rpy="0 0 0"/>
+  </xacro:teledyne_wayfinder_dvl_macro>
+  <!-- Sonar (Ping360 scanning imaging sonar) -->
+  <xacro:ping360_bluerobotics namespace="${namespace}" parent_link="${namespace}/base_link" suffix="_ping360" >
+    <origin xyz="0.22 0 -0.0" rpy="0 ${40*pi/180} 0"/>
+  </xacro:ping360_bluerobotics>
   <!-- Mount a GPS. -->
   <xacro:default_gps namespace="${namespace}" parent_link="${namespace}/base_link" />

File: bluerov2/bluerov2_description/urdf/snippets.xacro (robot description, xacro)
@@ -84,4 +84,5 @@
     </gazebo>
   </xacro:macro>
+  <!-- raspberry pi CAMERA REV 1.3-->
   <xacro:macro name="bluerov_camera" params="namespace parent_link suffix *origin">
     <xacro:regular_camera_plugin_macro
@@ -92,9 +93,9 @@
       mass="0.001"
       update_rate="30"
-      hfov="1.5125"
+      hfov="0.93327"
       width="1920"
       height="1080"
       stddev="0.01"
-      scale="1.0">
+      scale="0.001">
       <inertia ixx="0.00001" ixy="0.0" ixz="0.0" iyy="0.00001" iyz="0.0" izz="0.00001" />
       <xacro:insert_block name="origin" />

File: uuv_simulator/uuv_sensor_plugins/uuv_sensor_ros_plugins/urdf/camera_snippets.xacro (robot description, xacro)
@@ -34,5 +34,5 @@
       height="492"
       stddev="0.02"
-      scale="1.0">
+      scale="0.0001">
       <inertia ixx="0.00001" ixy="0.0" ixz="0.0" iyy="0.00001" iyz="0.0" izz="0.00001" />
       <xacro:insert_block name="origin" />
@@ -53,5 +53,5 @@
       scale="1.0">
       <inertia ixx="0.00001" ixy="0.0" ixz="0.0" iyy="0.00001" iyz="0.0" izz="0.00001" />
-      <xacro:insert_block name="origin" />>
+      <xacro:insert_block name="origin" />
     </xacro:regular_camera_plugin_macro>
   </xacro:macro>
@@ -69,5 +69,5 @@
       <visual>
         <geometry>
-          <mesh filename="file://$(find uuv_sensor_ros_plugins)/meshes/oe14-372.dae" scale="${scale} ${scale} ${scale}"/>
+          <mesh filename="file://$(find uuv_sensor_ros_plugins)/meshes/bluerov2_camera.dae" scale="${scale} ${scale} ${scale}"/>
         </geometry>
       </visual>

File: uuv_simulator/uuv_sensor_plugins/uuv_sensor_ros_plugins/urdf/sensor_snippets.xacro (robot description, xacro)
@@ -19,8 +19,11 @@
   <xacro:include filename="$(find uuv_sensor_ros_plugins)/urdf/dvl_snippets.xacro" />
   <xacro:include filename="$(find uuv_sensor_ros_plugins)/urdf/rpt_snippets.xacro" />
-  <xacro:include filename="$(find uuv_sensor_ros_plugins)/urdf/sonar_snippets.xacro" />
+  <!--<xacro:include filename="$(find uuv_sensor_ros_plugins)/urdf/sonar_snippets.xacro" /> -->
   <xacro:include filename="$(find uuv_sensor_ros_plugins)/urdf/stereo_snippets.xacro" />
   <xacro:include filename="$(find uuv_sensor_ros_plugins)/urdf/gps_sensor_snippets.xacro" />
   <xacro:include filename="$(find uuv_sensor_ros_plugins)/urdf/pose_3d_snippets.xacro" />
   <xacro:include filename="$(find uuv_sensor_ros_plugins)/urdf/chemical_concentration_snippets.xacro"/>
+  <xacro:include filename="$(find uuv_sensor_ros_plugins)/urdf/teledyne_wayfinderDVL.xacro"/>
+  <xacro:include filename="$(find uuv_sensor_ros_plugins)/urdf/multibeam_sonar_snippets.xacro"/>
+  <xacro:include filename="$(find uuv_sensor_ros_plugins)/urdf/mechanical_scanning_sonar_snippets.xacro"/>
 </robot>
